File: aliceq.kicad_pcb (KiCad board)
At the start: 2 copper layers, 337.2 x 122.6 mm, 173 parts, among them J1 ISP-6, SW1 SW_Push, U1 ATmega32U4-AU, U2 PRTR5V0U2X, Y1 CLK

Commit message: progreso del fin de semana
Parts:
- added D80: LED_Small, LED_THT:LED_D1.8mm_W3.3mm_H2.4mm, F.Cu at (-13.2, 95.8)
- added D81: LED_Small, LED_THT:LED_D1.8mm_W3.3mm_H2.4mm, F.Cu at (-13.2, 100.3)
- added D82: LED_Small, LED_THT:LED_D1.8mm_W3.3mm_H2.4mm, F.Cu at (-13.2, 104.8)
- C1, C2, C3, C4, C5, C6: footprint Capacitor_SMD:C_0805_2012Metric_Pad1.15x1.40mm_HandSolder -> Capacitor_SMD:C_0603_1608Metric
- R1, R2, R3, R4, R5, R6: footprint Resistor_SMD:R_0805_2012Metric_Pad1.15x1.40mm_HandSolder -> Resistor_SMD:R_0603_1608Metric
- U1: value ATmega32U4-AU -> ATmega32U4-MU; footprint Package_QFP:TQFP-44_10x10mm_P0.8mm -> Package_DFN_QFN:QFN-44-1EP_7x7mm_P0.5mm_EP5.15x5.15mm
- USB1: footprint Type-C:HRO-TYPE-C-31-M-12-HandSoldering -> Type-C:HRO-TYPE-C-31-M-12-Assembly
- Y1: footprint Crystal:Crystal_SMD_3225-4Pin_3.2x2.5mm_HandSoldering -> Crystal:Crystal_SMD_3225-4Pin_3.2x2.5mm
- moved SW1 349.3 mm to (182.9, 14.6)
- moved F1 320.9 mm to (150.8, 21.5), turned to 90 degrees
- moved Y1 311.3 mm to (154.2, 76.2), turned to 45 degrees
- moved J1 308.4 mm to (170.4, 13.9), turned to 90 degrees
- moved R5 297.3 mm to (149.2, 15.0)
- moved C1 294.7 mm to (152.7, 65.6), turned to -135 degrees
- moved C7 282.6 mm to (156.1, 79.5), turned to 135 degrees
- moved C8 277.1 mm to (157.6, 78.0), turned to 135 degrees
- moved C5 275.3 mm to (153.7, 67.3), turned to 45 degrees
- moved C2 275.1 mm to (156.6, 73.0), turned to -135 degrees
- moved R1 273.7 mm to (141.4, 73.0), turned to -45 degrees
- moved R4 273.5 mm to (160.1, 15.0), turned to 0 degrees
- moved R6 266.6 mm to (176.9, 16.4)
- moved D68 245.7 mm to (250.1, 142.9)
- moved D73 245.2 mm to (232.6, 136.2)
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Connections:
- net Net-(R2-Pad1) renamed DN
- net Net-(R3-Pad2) renamed DP
- U1 pad 30: ROW1 -> ROW4
- U1 pad 41: unconnected-(U1-Pad41) -> ROW1
Routing:
- net ROW3: track 0.00 -> 351.3 mm
- net ROW1: track 0.00 -> 338.9 mm, vias 0 -> 2
- net ROW2: track 0.00 -> 333.4 mm
- net ROW4: track 0.00 -> 330.9 mm
- net ROW0: track 0.00 -> 323.1 mm, vias 0 -> 3
- net +5V: track 0.00 -> 136.9 mm, vias 0 -> 6
- net COL1: track 0.00 -> 108.6 mm
- net GND: track 0.00 -> 104.7 mm, vias 0 -> 2
- net COL7: track 0.00 -> 102.8 mm
- net COL10: track 0.00 -> 97.0 mm
- net COL6: track 0.00 -> 92.4 mm
- net COL14: track 0.00 -> 92.2 mm
- net COL5: track 0.00 -> 91.7 mm
- net COL3: track 0.00 -> 89.9 mm
- net COL13: track 0.00 -> 88.2 mm
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- added copper zone on B.Cu, net GND
- added copper zone on F.Cu, net GND
Other:
- outline, holes or cut-outs redrawn

Commit message: Terminado el ruteado, faltan los leds y el RGB
Parts:
- added D83: WS2812B, LED_SMD:LED_WS2812B_PLCC4_5.0x5.0mm_P3.2mm, B.Cu at (58.1, 118.1)
- added D84: WS2812B, LED_SMD:LED_WS2812B_PLCC4_5.0x5.0mm_P3.2mm, B.Cu at (5.30, 111.6)
- added D85: WS2812B, LED_SMD:LED_WS2812B_PLCC4_5.0x5.0mm_P3.2mm, B.Cu at (1.00, 87.7)
- added D86: WS2812B, LED_SMD:LED_WS2812B_PLCC4_5.0x5.0mm_P3.2mm, B.Cu at (-1.30, 60.6)
- added D87: WS2812B, LED_SMD:LED_WS2812B_PLCC4_5.0x5.0mm_P3.2mm, B.Cu at (-0.15, 32.6)
- added D88: WS2812B, LED_SMD:LED_WS2812B_PLCC4_5.0x5.0mm_P3.2mm, B.Cu at (25.2, 29.4)
- added D93: WS2812B, LED_SMD:LED_WS2812B_PLCC4_5.0x5.0mm_P3.2mm, B.Cu at (132.2, 31.6)
- added D94: WS2812B, LED_SMD:LED_WS2812B_PLCC4_5.0x5.0mm_P3.2mm, B.Cu at (84.4, 29.4)
- moved D71 155.0 mm to (324.4, 31.2)
- moved D74 144.3 mm to (100.0, 118.1)
- moved D72 130.3 mm to (324.6, 53.3)
- moved D70 126.5 mm to (282.7, 28.9)
- moved D68 120.3 mm to (210.7, 29.3)
- moved D73 108.0 mm to (325.4, 81.0)
- moved D69 107.1 mm to (243.0, 29.3)
- moved D75 103.9 mm to (137.2, 131.0)
- moved D78 82.8 mm to (286.7, 112.8)
- moved D79 76.2 mm to (326.1, 106.9)
- moved D77 39.2 mm to (252.3, 114.5)
- moved D76 23.9 mm to (219.2, 123.9)
- moved R4 17.2 mm to (168.2, 30.1)
- moved R5 17.2 mm to (157.3, 30.1)
- moved U2 17.2 mm to (162.7, 32.9)
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Connections:
- D74 pad 2: unconnected-(D74-Pad2) -> Net-(D74-Pad2)
- U1 pad 18: COL10 -> COL9
- U1 pad 19: COL11 -> COL8
- U1 pad 20: COL12 -> COL7
- U1 pad 21: COL13 -> COL10
- U1 pad 22: COL14 -> COL11
- U1 pad 25: COL7 -> COL12
- U1 pad 26: COL8 -> COL13
- U1 pad 27: COL9 -> COL14
- U1 pad 28: ROW3 -> ROW4
- U1 pad 29: ROW2 -> ROW3
- U1 pad 30: ROW4 -> ROW2
- U1 pad 31: COL1 -> COL5
- U1 pad 32: COL0 -> COL6
- U1 pad 36: COL2 -> COL4
- U1 pad 38: COL4 -> COL2
- U1 pad 39: COL5 -> COL1
- U1 pad 40: COL6 -> COL0
Routing:
- net COL14: track 92.2 -> 281.7 mm, vias 0 -> 2
- net COL13: track 88.2 -> 259.4 mm, vias 0 -> 3
- net COL0: track 73.6 -> 234.1 mm
- net COL12: track 71.1 -> 220.4 mm, vias 0 -> 3
- net COL1: track 108.6 -> 238.2 mm, vias 0 -> 1
- net COL11: track 73.4 -> 202.9 mm, vias 0 -> 3
- net COL2: track 86.3 -> 191.9 mm, vias 0 -> 1
- net COL10: track 97.0 -> 195.7 mm, vias 0 -> 3
- net COL3: track 89.9 -> 173.2 mm, vias 0 -> 1
- net COL9: track 72.5 -> 138.7 mm, vias 0 -> 3
- net COL4: track 67.9 -> 130.0 mm, vias 0 -> 1
- net ROW4: track 330.9 -> 377.9 mm, vias 0 -> 2
- net COL8: track 72.9 -> 119.4 mm, vias 0 -> 3
- net COL5: track 91.7 -> 131.2 mm, vias 0 -> 1
- net ROW1: track 338.9 -> 376.5 mm
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Other:
- board size 337.2 x 122.6 mm -> 337.2 x 123.2 mm
