File: aliceq.kicad_sch (KiCad schematic)
At the start: 184 parts, among them J1 ISP-6, SW1 SW_Push, U1 ATmega32U4-AU, U2 PRTR5V0U2X, Y1 CLK

Commit message: Fixing hotswap socket positioning
Parts:
- MX32: footprint MX_Only:MXOnly-1U-Hotswap -> MX_Only:MXOnly-1.25U-Hotswap
- MX71: footprint MX_Only:MXOnly-2.75U-Hotswap-ReversedStabilizers -> MX_Only:MXOnly-2.75U-Hotswap
